Commit message: ball chaser bugs fixed

File: catkin_ws/src/my_robot/urdf/my_robot.xacro (robot description, xacro)
@@ -69,5 +69,5 @@
       <origin xyz="0 0 0" rpy="0 1.5707 1.5707"/>
       <geometry>
-        <cylinder radius="0.2" length="0.05"/>
+        <cylinder radius="0.1" length="0.1"/>
       </geometry>
     </collision>
@@ -75,5 +75,5 @@
       <origin xyz="0 0 0" rpy="0 1.5707 1.5707"/>
       <geometry>
-        <cylinder radius="0.2" length="0.05"/>
+        <cylinder radius="0.1" length="0.1"/>
       </geometry>
     </visual>
@@ -92,5 +92,5 @@
       <origin xyz="0 0 0" rpy="0 1.5707 1.5707"/>
       <geometry>
-        <cylinder radius="0.2" length="0.05"/>
+        <cylinder radius="0.1" length="0.1"/>
       </geometry>
     </collision>
@@ -98,5 +98,5 @@
       <origin xyz="0 0 0" rpy="0 1.5707 1.5707"/>
       <geometry>
-        <cylinder radius="0.2" length="0.05"/>
+        <cylinder radius="0.1" length="0.1"/>
       </geometry>
     </visual>
