Commit message: re-packaged project2 submission

File: Project2Submission/my_robot/urdf/my_robot.xacro (robot description, xacro)
@@ -69,5 +69,5 @@
       <origin xyz="0 0 0" rpy="0 1.5707 1.5707"/>
       <geometry>
-        <cylinder radius="0.1" length="0.05"/>
+        <cylinder radius="0.1" length="0.1"/>
       </geometry>
     </collision>
@@ -75,5 +75,5 @@
       <origin xyz="0 0 0" rpy="0 1.5707 1.5707"/>
       <geometry>
-        <cylinder radius="0.1" length="0.05"/>
+        <cylinder radius="0.1" length="0.1"/>
       </geometry>
     </visual>
@@ -92,5 +92,5 @@
       <origin xyz="0 0 0" rpy="0 1.5707 1.5707"/>
       <geometry>
-        <cylinder radius="0.1" length="0.05"/>
+        <cylinder radius="0.1" length="0.1"/>
       </geometry>
     </collision>
@@ -98,5 +98,5 @@
       <origin xyz="0 0 0" rpy="0 1.5707 1.5707"/>
       <geometry>
-        <cylinder radius="0.1" length="0.05"/>
+        <cylinder radius="0.1" length="0.1"/>
       </geometry>
     </visual>
@@ -179,3 +179,9 @@
     <material>Gazebo/Green</material>
   </gazebo>
+  <gazebo reference="right_wheel">
+    <material>Gazebo/Green</material>
+  </gazebo>
+  <gazebo reference="chassis">
+    <material>Gazebo/Orange</material>
+  </gazebo>
 </robot>
