Commit message: Improve localisation. Map now has doorways and is in the same orientation as gazebo world

File: project4/catkin_ws/src/my_robot/urdf/my_robot.xacro (robot description, xacro)
@@ -22,5 +22,5 @@
       <origin xyz="0 0 0" rpy=" 0 0 0"/>
       <geometry>
-        <box size=".4 .2 .1"/>
+        <box size=".3 .2 .1"/>
       </geometry>
     </collision>
@@ -28,5 +28,5 @@
       <origin xyz="0 0 0" rpy=" 0 0 0"/>
       <geometry>
-        <box size=".4 .2 .1"/>
+        <box size=".3 .2 .1"/>
       </geometry>
     </visual>
@@ -69,5 +69,5 @@
       <origin xyz="0 0 0" rpy="0 1.5707 1.5707"/>
       <geometry>
-        <cylinder radius="0.1" length="0.1"/>
+        <cylinder radius="0.1" length="0.05"/>
       </geometry>
     </collision>
@@ -75,5 +75,5 @@
       <origin xyz="0 0 0" rpy="0 1.5707 1.5707"/>
       <geometry>
-        <cylinder radius="0.1" length="0.1"/>
+        <cylinder radius="0.1" length="0.05"/>
       </geometry>
     </visual>
@@ -92,5 +92,5 @@
       <origin xyz="0 0 0" rpy="0 1.5707 1.5707"/>
       <geometry>
-        <cylinder radius="0.1" length="0.1"/>
+        <cylinder radius="0.1" length="0.05"/>
       </geometry>
     </collision>
@@ -98,5 +98,5 @@
       <origin xyz="0 0 0" rpy="0 1.5707 1.5707"/>
       <geometry>
-        <cylinder radius="0.1" length="0.1"/>
+        <cylinder radius="0.1" length="0.05"/>
       </geometry>
     </visual>

Commit message: Feat - Add depth camera to my_robot

File: project4/catkin_ws/src/my_robot/urdf/my_robot.xacro (robot description, xacro)
@@ -176,4 +176,11 @@
     <axis xyz="0 1 0" rpy="0 0 0"/>
   </joint>
+  <joint name="camera_optical_joint" type="fixed">
+    <origin xyz="0 0 0" rpy="-1.5707 0 -1.5707"/>
+    <parent link="camera"/>
+    <child link="camera_link_optical"/>
+  </joint>
+  <link name="camera_link_optical">
+  </link>
   <gazebo reference="left_wheel">
     <material>Gazebo/Green</material>

Commit message: Bug - Eliminate transform bug in robot urdf.

File: project4/catkin_ws/src/my_robot/urdf/my_robot.xacro (robot description, xacro)
@@ -118,5 +118,5 @@
     <dynamics damping="1.0" friction="1.0"/>
   </joint>
-  <link name="camera">
+  <link name="camera_link">
     <inertial>
       <mass value="0.1"/>
@@ -143,5 +143,5 @@
   <joint type="fixed" name="camera_joint">
     <origin xyz="0.2 0 0" rpy="0 0 0"/>
-    <child link="camera"/>
+    <child link="camera_link"/>
     <parent link="chassis"/>
     <axis xyz="0 1 0" rpy="0 0 0"/>
@@ -178,5 +178,5 @@
   <joint name="camera_optical_joint" type="fixed">
     <origin xyz="0 0 0" rpy="-1.5707 0 -1.5707"/>
-    <parent link="camera"/>
+    <parent link="camera_link"/>
     <child link="camera_link_optical"/>
   </joint>
